Commit message: Added simulation

File: src/simulation/urdf/ribbit.urdf (robot description, URDF)
Before this commit: robot ribbit, 15 links, 7 joints
Links:
- removed link hokuyo_link
- removed link primesense_link
- added link camera_link; visual box size=0.0 0.0 0.0
- added link laser_link; visual box size=0.0 0.0 0.0
Joints:
- removed joint hokuyo_joint
- removed joint primesense_joint
- added joint camera_joint: type fixed, parent base_link, child camera_link, origin xyz=0. 0. 0. rpy=0. 0. 0.
- added joint laser_joint: type fixed, parent base_link, child laser_link, origin xyz=0. 0. 0. rpy=0. 0. 0.
