Commit message: Removed sonar

File: simulation/urdf/simulation.urdf (robot description, URDF)
Before this commit: robot simulation, 6 links, 5 joints
Links:
- removed link sonar_down_link
- removed link sonar_up_link
Joints:
- removed joint sonar_down_joint
- removed joint sonar_up_joint

Commit message: Changed from dd_slam_link to base_link

File: simulation/urdf/simulation.urdf (robot description, URDF)
Before this commit: robot simulation, 4 links, 3 joints
Links:
- removed link dd_slam_link
- added link base_link
Joints:
- joint camera_joint: parent dd_slam_link -> base_link
- joint laser_joint: parent dd_slam_link -> base_link
- joint teraranger_joint: parent dd_slam_link -> base_link
