Commit message: Created xacro models instead

File: simulation/urdf/model.urdf (robot description, URDF)
Before this commit: robot iris, 8 links, 7 joints
Links:
- link camera_link: geometry visual mesh filename=package://simulation/urdf/meshes/r200/r200.dae scale=1.0 1.0 1.0
- link rotor_0: geometry visual mesh filename=package://px4/Tools/sitl_gazebo/models/rotors_description/m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 scale=1 1 1
- link rotor_1: geometry visual mesh filename=package://px4/Tools/sitl_gazebo/models/rotors_description/m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 scale=1 1 1
- link rotor_2: geometry visual mesh filename=package://px4/Tools/sitl_gazebo/models/rotors_description/m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 scale=1 1 1
- link rotor_3: geometry visual mesh filename=package://px4/Tools/sitl_gazebo/models/rotors_description/m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 scale=1 1 1
Joints:
- joint rotor_0_joint: type fixed -> revolute
- joint rotor_1_joint: type fixed -> revolute
- joint rotor_2_joint: type fixed -> revolute
- joint rotor_3_joint: type fixed -> revolute

File: simulation/xacro/multirotor.urdf.xacro (robot description, xacro)
@@ -45,63 +45,5 @@
     </collision>
   </link>
-  <link name="${namespace}/rgbd_link">
-    <gravity>0</gravity>
-    <kinematic>0</kinematic>
-    <visual name="visual">
-      <geometry>
-        <mesh filename="model://kinect/meshes/kinect.dae" scale="1 1 1" />
-      </geometry>
-    </visual>
-    <inertial>
-      <!-- [kg] -->
-      <mass value="0.05" />
-      <origin xyz="0 0 0" />
-      <inertia ixx="0.07" ixy="0.0" ixz="0.0" iyy="0.08" iyz="0.0" izz="0.12" />
-    </inertial>
-  </link>
-  <gazebo reference="${namespace}/rgbd_link">
-    <sensor type="depth" name="rgbd">
-      <always_on>1</always_on>
-      <visualize>false</visualize>
-      <update_rate>6.0</update_rate>
-      <camera>
-        <horizontal_fov>2.00712864</horizontal_fov>
-        <image>
-          <width>424</width>
-          <height>240</height>
-          <format>R8G8B8</format>
-        </image>
-        <depth_camera>
-        </depth_camera>
-        <clip>
-          <near>0.1</near>
-          <far>100</far>
-        </clip>
-      </camera>
-      <plugin name="${namespace}_rgbd_controller" filename="libgazebo_ros_depth_camera.so">        <!-- libgazebo_ros_depth_camera.so -->
-        <alwaysOn>true</alwaysOn>
-        <updateRate>6.0</updateRate>
-        <cameraName>camera</cameraName>
-        <frameName>/${namespace}_rgbd_link</frameName>
-        <imageTopicName>rgb/image_raw</imageTopicName>
-        <depthImageTopicName>depth/image_raw</depthImageTopicName>
-        <pointCloudTopicName>depth/points</pointCloudTopicName>
-        <cameraInfoTopicName>rgb/camera_info</cameraInfoTopicName>
-        <depthImageCameraInfoTopicName>depth/camera_info</depthImageCameraInfoTopicName>
-        <pointCloudCutoff>0.1</pointCloudCutoff>
-        <pointCloudCutoffMax>7.0</pointCloudCutoffMax>
-        <hackBaseline>0.07</hackBaseline>
-        <distortionK1>0.0</distortionK1>
-        <distortionK2>0.0</distortionK2>
-        <distortionK3>0.0</distortionK3>
-        <distortionT1>0.0</distortionT1>
-        <distortionT2>0.0</distortionT2>
-        <CxPrime>0.0</CxPrime>
-        <Cx>0.0</Cx>
-        <Cy>0.0</Cy>
-        <focalLength>0.0</focalLength>
-      </plugin>
-    </sensor>
-  </gazebo>
+  <!-- Sensors -->
   <joint name='${namespace}/rgbd_joint' type='fixed'>
     <child link="${namespace}/rgbd_link" />
